File: hardware/main-board/main-board-input.sch (KiCad schematic (older format))
At the start: 36 parts, among them J4 Blackout Switch, SW1 Start, SW10 Menu, SW11 Rotary Encoder, SW2 Focus, SW3 Inc Exposure, SW4 Dec Exposure, SW5 Inc Contrast, SW6 Dec Contrast, SW7 Test Strip, SW8 Add Adjustment, SW9 Cancel, U7 TCA8418, U8 STP16CPC26

Commit message: Schematic cleanup
Other:
- note added: "All LEDs used in this section must emit at wavelengths\noutside the sensitivity of B&W printing paper"
- note added: "Display & Indicator Shutoff Switch"
- note added: "Enlarger Control Buttons"
- note added: "Exposure Adjustment Buttons"
- note added: "J4 is a connector that connects to\na panel mounted rocker switch"
- note added: "Menu & Mode Select Buttons"
- note added: "R8 sets the LED current\nat approximately 5mA"
- note added: "Value Adjustment Knob"
- note removed: "J4 is a wire-to-board connection from\na panel mounted rocker switch"
- note removed: "Need to do darkroom testing of all LED choices for this."
- moved on the sheet: C28, C29, D10, D3, D4, D5, D6, D7, D8, D9, J4, R21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

Commit message: Added "User Label" field to clean up BOM data for labeled common parts
This change is to prevent things like buttons, connectors, and relays
from being ungrouped on the BOM.
Parts:
- J4: value Blackout Switch -> Conn_01x02; User Label (none) -> Blackout Switch
- SW1: value Start -> SW_Push_Long; User Label (none) -> Start
- SW10: value Menu -> SW_Push_LED; User Label (none) -> Menu
- SW11: value Rotary Encoder -> Rotary_Encoder_Switch; User Label (none) -> Rotary Encoder
- SW2: value Focus -> SW_Push_Long; User Label (none) -> Focus
- SW3: value Inc Exposure -> SW_Push; User Label (none) -> Inc Exposure
- SW4: value Dec Exposure -> SW_Push; User Label (none) -> Dec Exposure
- SW5: value Inc Contrast -> SW_Push; User Label (none) -> Inc Contrast
- SW6: value Dec Contrast -> SW_Push; User Label (none) -> Dec Contrast
- SW7: value Test Strip -> SW_Push_LED; User Label (none) -> Test Strip
- SW8: value Add Adjustment -> SW_Push_LED; User Label (none) -> Add Adjustment
- SW9: value Cancel -> SW_Push_LED; User Label (none) -> Cancel
