File: hardware/main-board/main-board-power.kicad_sch (KiCad schematic)
At the start: 39 parts, among them J3 Power Board, J4 DMX512, U4 RT8258, U5 RT8258

Commit message: Remove main board test points
The power test points were minimally useful, and the part currently
being used for them was causing clearance issues with the display. While
these could have been replaced with pads or SMD test points, it was
simply easier to just remove them for now.

Refs #43
Parts:
- removed TP1, TP2, TP3, TP4: TestPoint, TestPoint:TestPoint_Keystone_5005-5009_Compact, symbol Connector:TestPoint
Changed lines of the file:
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@@
-    )
-  )
-  (symbol (lib_id "Connector:TestPoint") (at 191.135 62.865 270) (unit 1)
-    (in_bom yes) (on_board yes) (dnp no)
-    (property "Reference" "TP3" (at 196.215 62.865 90)
-      (effects (font (size 1.27 1.27)) (justify left))
-    )
-    (property "Value" "TestPoint" (at 194.1068 61.3918 0)
-      (effects (font (size 1.27 1.27)) (justify right) hide)
-    )
-    (property "Footprint" "TestPoint:TestPoint_Keystone_5005-5009_Compact" (at 191.135 67.945 0)
-      (effects (font (size 1.27 1.27)) hide)
-    )
-    (property "Datasheet" "http://www.keyelco.com/product-pdf.cfm?p=1314" (at 191.135 67.945 0)
-      (effects (font (size 1.27 1.27)) hide)
-    )
-    (property "Description" "PC TEST POINT COMPACT BLACK" (at 191.135 62.865 0)
-      (effects (font (size 1.27 1.27)) hide)
-    )
-    (property "Manufacturer" "Keystone Electronics" (at 191.135 62.865 0)
-      (effects (font (size 1.27 1.27)) hide)
-    )
-    (property "Manufacturer PN" "5006" (at 191.135 62.865 0)
-      (effects (font (size 1.27 1.27)) hide)
-    )
-    (property "Supplier" "Digi-Key" (at 191.135 62.865 0)
-      (effects (font (size 1.27 1.27)) hide)
-    )
-    (property "Supplier PN" "36-5006-ND" (at 191.135 62.865 0)
-      (effects (font (size 1.27 1.27)) hide)
-    )
-    (pin "1")
-    (instances
-      (project "main-board"
-        (path "/31a301d9-d769-4a35-943a-fe3e3609e773/00000000-0000-0000-0000-00005f8b674d"
-          (reference "TP3") (unit 1)
-        )
-      )
     )
   )
@@
     )
   )
-  (symbol (lib_id "power:GND") (at 74.93 31.115 0) (unit 1)
-    (in_bom yes) (on_board yes) (dnp no)
-    (property "Reference" "#PWR045" (at 74.93 37.465 0)
-      (effects (font (size 1.27 1.27)) hide)
-    )
-    (property "Value" "GND" (at 74.93 34.925 0)
-      (effects (font (size 1.27 1.27)))
-    )
-    (property "Footprint" "" (at 74.93 31.115 0)
-      (effects (font (size 1.27 1.27)) hide)
-    )
-    (property "Datasheet" "" (at 74.93 31.115 0)
-      (effects (font (size 1.27 1.27)) hide)
-    )
-    (pin "1")
-    (instances
-      (project "main-board"
-        (path "/31a301d9-d769-4a35-943a-fe3e3609e773/00000000-0000-0000-0000-00005f8b674d"
-          (reference "#PWR045") (unit 1)
-        )
-      )
-    )
-  )
   (symbol (lib_id "power:+5V") (at 191.135 100.33 0) (unit 1)
     (in_bom yes) (on_board yes) (dnp no) (fields_autoplaced)
@@
     )
   )
-  (symbol (lib_id "power:+12V") (at 69.215 31.115 0) (unit 1)
-    (in_bom yes) (on_board yes) (dnp no)
-    (property "Reference" "#PWR042" (at 69.215 34.925 0)
-      (effects (font (size 1.27 1.27)) hide)
-    )
-    (property "Value" "+12V" (at 69.596 26.7208 0)
-      (effects (font (size 1.27 1.27)))
-    )
-    (property "Footprint" "" (at 69.215 31.115 0)
-      (effects (font (size 1.27 1.27)) hide)
-    )
-    (property "Datasheet" "" (at 69.215 31.115 0)
-      (effects (font (size 1.27 1.27)) hide)
-    )
-    (pin "1")
-    (instances
-      (project "main-board"
-        (path "/31a301d9-d769-4a35-943a-fe3e3609e773/00000000-0000-0000-0000-00005f8b674d"
-          (reference "#PWR042") (unit 1)
-        )
-      )
-    )
-  )
   (symbol (lib_id "Device:R_Small") (at 139.065 106.68 0) (unit 1)
     (in_bom yes) (on_board yes) (dnp no) (fields_autoplaced)
@@
         (path "/e1031c6b-0ca1-4aad-ab4f-7f9003f9770e"
           (reference "C?") (unit 1)
-        )
-      )
-    )
-  )
-  (symbol (lib_id "Connector:TestPoint") (at 191.135 102.235 270) (unit 1)
-    (in_bom yes) (on_board yes) (dnp no)
-    (property "Reference" "TP4" (at 196.215 102.235 90)
-      (effects (font (size 1.27 1.27)) (justify left))
-    )
-    (property "Value" "TestPoint" (at 194.1068 100.7618 0)
-      (effects (font (size 1.27 1.27)) (justify right) hide)
-    )
-    (property "Footprint" "TestPoint:TestPoint_Keystone_5005-5009_Compact" (at 191.135 107.315 0)
-      (effects (font (size 1.27 1.27)) hide)
-    )
-    (property "Datasheet" "http://www.keyelco.com/product-pdf.cfm?p=1314" (at 191.135 107.315 0)
-      (effects (font (size 1.27 1.27)) hide)
-    )
-    (property "Description" "PC TEST POINT COMPACT BLACK" (at 191.135 102.235 0)
-      (effects (font (size 1.27 1.27)) hide)
-    )
-    (property "Manufacturer" "Keystone Electronics" (at 191.135 102.235 0)
-      (effects (font (size 1.27 1.27)) hide)
-    )
-    (property "Manufacturer PN" "5006" (at 191.135 102.235 0)
-      (effects (font (size 1.27 1.27)) hide)
-    )
-    (property "Supplier" "Digi-Key" (at 191.135 102.235 0)
-      (effects (font (size 1.27 1.27)) hide)
-    )
-    (property "Supplier PN" "36-5006-ND" (at 191.135 102.235 0)
-      (effects (font (size 1.27 1.27)) hide)
-    )
-    (pin "1")
-    (instances
-      (project "main-board"
-        (path "/31a301d9-d769-4a35-943a-fe3e3609e773/00000000-0000-0000-0000-00005f8b674d"
-          (reference "TP4") (unit 1)
         )
       )
@@
     )
   )
-  (symbol (lib_id "Connector:TestPoint") (at 69.215 31.115 180) (unit 1)
-    (in_bom yes) (on_board yes) (dnp no)
-    (property "Reference" "TP1" (at 67.7418 32.9438 0)
-      (effects (font (size 1.27 1.27)) (justify left))
-    )
-    (property "Value" "TestPoint" (at 70.6882 34.0868 0)
-      (effects (font (size 1.27 1.27)) (justify right) hide)
-    )
-    (property "Footprint" "TestPoint:TestPoint_Keystone_5005-5009_Compact" (at 64.135 31.115 0)
-      (effects (font (size 1.27 1.27)) hide)
-    )
-    (property "Datasheet" "http://www.keyelco.com/product-pdf.cfm?p=1314" (at 64.135 31.115 0)
-      (effects (font (size 1.27 1.27)) hide)
-    )
-    (property "Description" "PC TEST POINT COMPACT BLACK" (at 69.215 31.115 0)
-      (effects (font (size 1.27 1.27)) hide)
-    )
-    (property "Manufacturer" "Keystone Electronics" (at 69.215 31.115 0)
-      (effects (font (size 1.27 1.27)) hide)
-    )
-    (property "Manufacturer PN" "5006" (at 69.215 31.115 0)
-      (effects (font (size 1.27 1.27)) hide)
-    )
-    (property "Supplier" "Digi-Key" (at 69.215 31.115 0)
-      (effects (font (size 1.27 1.27)) hide)
-    )
-    (property "Supplier PN" "36-5006-ND" (at 69.215 31.115 0)
-      (effects (font (size 1.27 1.27)) hide)
-    )
-    (pin "1")
-    (instances
-      (project "main-board"
-        (path "/31a301d9-d769-4a35-943a-fe3e3609e773/00000000-0000-0000-0000-00005f8b674d"
-          (reference "TP1") (unit 1)
-        )
-      )
-    )
-  )
   (symbol (lib_id "Project:RT8258") (at 97.79 102.235 0) (unit 1)
     (in_bom yes) (on_board yes) (dnp no) (fields_autoplaced)
@@
         )
       )
-    )
-  )
-  (symbol (lib_id "Connector:TestPoint") (at 74.93 31.115 0) (unit 1)
-    (in_bom yes) (on_board yes) (dnp no)
-    (property "Reference" "TP2" (at 76.4032 29.2862 0)
-      (effects (font (size 1.27 1.27)) (justify left))
-    )
-    (property "Value" "TestPoint" (at 73.4568 28.1432 0)
-      (effects (font (size 1.27 1.27)) (justify right) hide)
-    )
-    (property "Footprint" "TestPoint:TestPoint_Keystone_5005-5009_Compact" (at 80.01 31.115 0)
-      (effects (font (size 1.27 1.27)) hide)
-    )
-    (property "Datasheet" "http://www.keyelco.com/product-pdf.cfm?p=1314" (at 80.01 31.115 0)
-      (effects (font (size 1.27 1.27)) hide)
-    )
-    (property "Description" "PC TEST POINT COMPACT BLACK" (at 74.93 31.115 0)
-      (effects (font (size 1.27 1.27)) hide)
-    )
-    (property "Manufacturer" "Keystone Electronics" (at 74.93 31.115 0)
-      (effects (font (size 1.27 1.27)) hide)
-    )
-    (property "Manufacturer PN" "5006" (at 74.93 31.115 0)
-      (effects (font (size 1.27 1.27)) hide)
-    )
-    (property "Supplier" "Digi-Key" (at 74.93 31.115 0)
-      (effects (font (size 1.27 1.27)) hide)
-    )
-    (property "Supplier PN" "36-5006-ND" (at 74.93 31.115 0)
-      (effects (font (size 1.27 1.27)) hide)
-    )
-    (pin "1")
-    (instances
-      (project "main-board"
-        (path "/31a301d9-d769-4a35-943a-fe3e3609e773/00000000-0000-0000-0000-00005f8b674d"
-          (reference "TP2") (unit 1)
-        )
-      )
