File: hardware/meter-probe-tsl2521/meter-probe-tsl2521.kicad_sch (KiCad schematic)
At the start: 44 parts, among them J1 Cable, J2 Cable, SW1 Sensor Button, U1 TSL2521, U2 M24C02-D, U3 PCA9527, U4 TC1301A-APA, U5 USBLC6-2SC6, U6 TCA9801

Commit message: Fill in missing BOM data on meter probe variant
Parts:
- U1: Manufacturer (none) -> ams OSRAM; Manufacturer PN (none) -> TSL25213M; Supplier (none) -> Digi-Key; Supplier PN (none) -> 4991-TSL25213MCT-ND
Changed lines of the file:
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@@
       (effects (font (size 1.27 1.27)) hide)
     )
-    (property "Description" "" (at 31.75 52.07 0)
+    (property "Description" "AMBIENT LIGHT SENSOR" (at 31.75 52.07 0)
       (effects (font (size 1.27 1.27)) hide)
     )
-    (property "Manufacturer" "" (at 31.75 52.07 0)
+    (property "Manufacturer" "ams OSRAM" (at 31.75 52.07 0)
       (effects (font (size 1.27 1.27)) hide)
     )
-    (property "Manufacturer PN" "" (at 31.75 52.07 0)
+    (property "Manufacturer PN" "TSL25213M" (at 31.75 52.07 0)
       (effects (font (size 1.27 1.27)) hide)
     )
-    (property "Supplier" "" (at 31.75 52.07 0)
+    (property "Supplier" "Digi-Key" (at 31.75 52.07 0)
       (effects (font (size 1.27 1.27)) hide)
     )
-    (property "Supplier PN" "" (at 31.75 52.07 0)
+    (property "Supplier PN" "4991-TSL25213MCT-ND" (at 31.75 52.07 0)
       (effects (font (size 1.27 1.27)) hide)
     )
