File: hardware/power-board/power-board.kicad_pcb (KiCad board)
At the start: 2 copper layers, 193 x 65 mm, 31 parts, among them J1 SW_SPST, J2 Main Board, J3 DMX512 Out Jack, J4 DMX512, K1 SPST-NO, K2 SPST-NO, P1 IEC320-C14, P2 IEC320-C13, P3 IEC320-C13, U1 SZNUD3124DMT1G, U2 THVD1439

Commit message: Update PCB data files to KiCad v8
This change involves the following:
- Opening and resaving all the files
- Adjusting the schematic connection grid to make ERC happy
- Updating various library symbols and footprints, where the changes
  entirely involve invisible metadata
Other:
- board text added: "ENLG"
- board text added: "Enlarger Power Output"
- board text added: "Mains Power Input"
- board text added: "SFLT"
- board text added: "Safelight Power Output"
- board text removed: "locked"

Commit message: Change power board mounting hole footprints
This changes them from the 3.2mm diameter M3 version to the
similar-looking 3.5mm diameter version. Position is still the same, and
the size isn't that different, but this should provide more flexibility
when rear panel alignment tolerances cause issue with the internal screw
holes lining up.

Fix #53
Parts:
- H1, H2: footprint MountingHole:MountingHole_3.2mm_M3_Pad_Via -> MountingHole:MountingHole_3.5mm_Pad_Via
Changed lines of the file:
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@@
 		)
 	)
-	(footprint "MountingHole:MountingHole_3.2mm_M3_Pad_Via"
+	(footprint "MountingHole:MountingHole_3.5mm_Pad_Via"
 		(layer "F.Cu")
 		(at 41 100)
-		(descr "Mounting Hole 3.2mm, M3")
-		(tags "mounting hole 3.2mm m3")
+		(descr "Mounting Hole 3.5mm")
+		(tags "mounting hole 3.5mm")
 		(property "Reference" "H1"
-			(at 0 -4.2 0)
+			(at 0 -4.5 0)
 			(layer "F.SilkS")
 			(hide yes)
@@
 		)
 		(property "Value" "MountingHole_Pad"
-			(at 0 4.2 0)
-			(layer "F.Fab")
-			(hide yes)
-			(effects
-				(font
-					(size 1 1)
-					(thickness 0.15)
-				)
-			)
-		)
-		(property "Footprint" "MountingHole:MountingHole_3.2mm_M3_Pad_Via"
+			(at 0 4.5 0)
+			(layer "F.Fab")
+			(effects
+				(font
+					(size 1 1)
+					(thickness 0.15)
+				)
+			)
+		)
+		(property "Footprint" "MountingHole:MountingHole_3.5mm_Pad_Via"
 			(at 0 0 0)
 			(unlocked yes)
@@
 		)
 		(property "Description" ""
-			(at 41 100 0)
+			(at 0 0 0)
+			(unlocked yes)
 			(layer "F.Fab")
 			(hide yes)
@@
 		(fp_circle
 			(center 0 0)
-			(end 3.2 0)
+			(end 3.5 0)
 			(stroke
 				(width 0.15)
@@
 		(fp_circle
 			(center 0 0)
-			(end 3.45 0)
+			(end 3.75 0)
 			(stroke
 				(width 0.05)
@@
 		)
 		(pad "1" thru_hole circle
-			(at -2.4 0)
-			(size 0.8 0.8)
-			(drill 0.5)
-			(layers "*.Cu" "*.Mask")
-			(remove_unused_layers no)
-			(net 9 "Earth")
-			(pinfunction "1")
-			(pintype "input")
-			(zone_connect 2)
-		)
-		(pad "1" thru_hole circle
-			(at -1.697056 -1.697056)
-			(size 0.8 0.8)
-			(drill 0.5)
-			(layers "*.Cu" "*.Mask")
-			(remove_unused_layers no)
-			(net 9 "Earth")
-			(pinfunction "1")
-			(pintype "input")
-			(zone_connect 2)
-		)
-		(pad "1" thru_hole circle
-			(at -1.697056 1.697056)
-			(size 0.8 0.8)
-			(drill 0.5)
-			(layers "*.Cu" "*.Mask")
-			(remove_unused_layers no)
-			(net 9 "Earth")
-			(pinfunction "1")
-			(pintype "input")
-			(zone_connect 2)
-		)
-		(pad "1" thru_hole circle
-			(at 0 -2.4)
+			(at -2.625 0)
+			(size 0.8 0.8)
+			(drill 0.5)
+			(layers "*.Cu" "*.Mask")
+			(remove_unused_layers no)
+			(net 9 "Earth")
+			(pinfunction "1")
+			(pintype "input")
+			(zone_connect 2)
+		)
+		(pad "1" thru_hole circle
+			(at -1.856155 -1.856155)
+			(size 0.8 0.8)
+			(drill 0.5)
+			(layers "*.Cu" "*.Mask")
+			(remove_unused_layers no)
+			(net 9 "Earth")
+			(pinfunction "1")
+			(pintype "input")
+			(zone_connect 2)
+		)
+		(pad "1" thru_hole circle
+			(at -1.856155 1.856155)
+			(size 0.8 0.8)
+			(drill 0.5)
+			(layers "*.Cu" "*.Mask")
+			(remove_unused_layers no)
+			(net 9 "Earth")
+			(pinfunction "1")
+			(pintype "input")
+			(zone_connect 2)
+		)
+		(pad "1" thru_hole circle
+			(at 0 -2.625)
 			(size 0.8 0.8)
 			(drill 0.5)
@@
 		(pad "1" thru_hole circle
 			(at 0 0)
-			(size 6.4 6.4)
-			(drill 3.2)
-			(layers "*.Cu" "*.Mask")
-			(remove_unused_layers no)
-			(net 9 "Earth")
-			(pinfunction "1")
-			(pintype "input")
-		)
-		(pad "1" thru_hole circle
-			(at 0 2.4)
-			(size 0.8 0.8)
-			(drill 0.5)
-			(layers "*.Cu" "*.Mask")
-			(remove_unused_layers no)
-			(net 9 "Earth")
-			(pinfunction "1")
-			(pintype "input")
-			(zone_connect 2)
-		)
-		(pad "1" thru_hole circle
-			(at 1.697056 -1.697056)
-			(size 0.8 0.8)
-			(drill 0.5)
-			(layers "*.Cu" "*.Mask")
-			(remove_unused_layers no)
-			(net 9 "Earth")
-			(pinfunction "1")
-			(pintype "input")
-			(zone_connect 2)
-		)
-		(pad "1" thru_hole circle
-			(at 1.697056 1.697056)
-			(size 0.8 0.8)
-			(drill 0.5)
-			(layers "*.Cu" "*.Mask")
-			(remove_unused_layers no)
-			(net 9 "Earth")
-			(pinfunction "1")
-			(pintype "input")
-			(zone_connect 2)
-		)
-		(pad "1" thru_hole circle
-			(at 2.4 0)
+			(size 7 7)
+			(drill 3.5)
+			(layers "*.Cu" "*.Mask")
+			(remove_unused_layers no)
+			(net 9 "Earth")
+			(pinfunction "1")
+			(pintype "input")
+		)
+		(pad "1" thru_hole circle
+			(at 0 2.625)
+			(size 0.8 0.8)
+			(drill 0.5)
+			(layers "*.Cu" "*.Mask")
+			(remove_unused_layers no)
+			(net 9 "Earth")
+			(pinfunction "1")
+			(pintype "input")
+			(zone_connect 2)
+		)
+		(pad "1" thru_hole circle
+			(at 1.856155 -1.856155)
+			(size 0.8 0.8)
+			(drill 0.5)
+			(layers "*.Cu" "*.Mask")
+			(remove_unused_layers no)
+			(net 9 "Earth")
+			(pinfunction "1")
+			(pintype "input")
+			(zone_connect 2)
+		)
+		(pad "1" thru_hole circle
+			(at 1.856155 1.856155)
+			(size 0.8 0.8)
+			(drill 0.5)
+			(layers "*.Cu" "*.Mask")
+			(remove_unused_layers no)
+			(net 9 "Earth")
+			(pinfunction "1")
+			(pintype "input")
+			(zone_connect 2)
+		)
+		(pad "1" thru_hole circle
+			(at 2.625 0)
 			(size 0.8 0.8)
 			(drill 0.5)
@@
 		)
 	)
-	(footprint "MountingHole:MountingHole_3.2mm_M3_Pad_Via"
+	(footprint "MountingHole:MountingHole_3.5mm_Pad_Via"
 		(layer "F.Cu")
 		(at 224 100)
-		(descr "Mounting Hole 3.2mm, M3")
-		(tags "mounting hole 3.2mm m3")
+		(descr "Mounting Hole 3.5mm")
+		(tags "mounting hole 3.5mm")
 		(property "Reference" "H2"
-			(at 0 -4.2 0)
+			(at 0 -4.5 0)
 			(layer "F.SilkS")
 			(hide yes)
@@
 		)
 		(property "Value" "MountingHole_Pad"
-			(at 0 4.2 0)
-			(layer "F.Fab")
-			(hide yes)
-			(effects
-				(font
-					(size 1 1)
-					(thickness 0.15)
-				)
-			)
-		)
-		(property "Footprint" "MountingHole:MountingHole_3.2mm_M3_Pad_Via"
+			(at 0 4.5 0)
+			(layer "F.Fab")
+			(effects
+				(font
+					(size 1 1)
+					(thickness 0.15)
+				)
+			)
+		)
+		(property "Footprint" "MountingHole:MountingHole_3.5mm_Pad_Via"
 			(at 0 0 0)
 			(unlocked yes)
@@
 		)
 		(property "Description" ""
-			(at 224 100 0)
+			(at 0 0 0)
+			(unlocked yes)
 			(layer "F.Fab")
 			(hide yes)
@@
 		(fp_circle
 			(center 0 0)
-			(end 3.2 0)
+			(end 3.5 0)
 			(stroke
 				(width 0.15)
@@
 		(fp_circle
 			(center 0 0)
-			(end 3.45 0)
+			(end 3.75 0)
 			(stroke
 				(width 0.05)
@@
 		)
 		(pad "1" thru_hole circle
-			(at -2.4 0)
-			(size 0.8 0.8)
-			(drill 0.5)
-			(layers "*.Cu" "*.Mask")
-			(remove_unused_layers no)
-			(net 9 "Earth")
-			(pinfunction "1")
-			(pintype "input")
-			(zone_connect 2)
-		)
-		(pad "1" thru_hole circle
-			(at -1.697056 -1.697056)
-			(size 0.8 0.8)
-			(drill 0.5)
-			(layers "*.Cu" "*.Mask")
-			(remove_unused_layers no)
-			(net 9 "Earth")
-			(pinfunction "1")
-			(pintype "input")
-			(zone_connect 2)
-		)
-		(pad "1" thru_hole circle
-			(at -1.697056 1.697056)
-			(size 0.8 0.8)
-			(drill 0.5)
-			(layers "*.Cu" "*.Mask")
-			(remove_unused_layers no)
-			(net 9 "Earth")
-			(pinfunction "1")
-			(pintype "input")
-			(zone_connect 2)
-		)
-		(pad "1" thru_hole circle
-			(at 0 -2.4)
+			(at -2.625 0)
+			(size 0.8 0.8)
+			(drill 0.5)
+			(layers "*.Cu" "*.Mask")
+			(remove_unused_layers no)
+			(net 9 "Earth")
+			(pinfunction "1")
+			(pintype "input")
+			(zone_connect 2)
+		)
+		(pad "1" thru_hole circle
+			(at -1.856155 -1.856155)
+			(size 0.8 0.8)
+			(drill 0.5)
+			(layers "*.Cu" "*.Mask")
+			(remove_unused_layers no)
+			(net 9 "Earth")
+			(pinfunction "1")
+			(pintype "input")
+			(zone_connect 2)
+		)
+		(pad "1" thru_hole circle
+			(at -1.856155 1.856155)
+			(size 0.8 0.8)
+			(drill 0.5)
+			(layers "*.Cu" "*.Mask")
+			(remove_unused_layers no)
+			(net 9 "Earth")
+			(pinfunction "1")
+			(pintype "input")
+			(zone_connect 2)
+		)
+		(pad "1" thru_hole circle
+			(at 0 -2.625)
 			(size 0.8 0.8)
 			(drill 0.5)
@@
 		(pad "1" thru_hole circle
 			(at 0 0)
-			(size 6.4 6.4)
-			(drill 3.2)
-			(layers "*.Cu" "*.Mask")
-			(remove_unused_layers no)
-			(net 9 "Earth")
-			(pinfunction "1")
-			(pintype "input")
-		)
-		(pad "1" thru_hole circle
-			(at 0 2.4)
-			(size 0.8 0.8)
-			(drill 0.5)
-			(layers "*.Cu" "*.Mask")
-			(remove_unused_layers no)
-			(net 9 "Earth")
-			(pinfunction "1")
-			(pintype "input")
-			(zone_connect 2)
-		)
-		(pad "1" thru_hole circle
-			(at 1.697056 -1.697056)
-			(size 0.8 0.8)
-			(drill 0.5)
-			(layers "*.Cu" "*.Mask")
-			(remove_unused_layers no)
-			(net 9 "Earth")
-			(pinfunction "1")
-			(pintype "input")
-			(zone_connect 2)
-		)
-		(pad "1" thru_hole circle
-			(at 1.697056 1.697056)
-			(size 0.8 0.8)
-			(drill 0.5)
-			(layers "*.Cu" "*.Mask")
-			(remove_unused_layers no)
-			(net 9 "Earth")
-			(pinfunction "1")
-			(pintype "input")
-			(zone_connect 2)
-		)
-		(pad "1" thru_hole circle
-			(at 2.4 0)
-			(size 0.8 0.8)
-			(drill 0.5)
+			(size 7 7)
+			(drill 3.5)
+			(layers "*.Cu" "*.Mask")
+			(remove_unused_layers no)
+			(net 9 "Earth")
+			(pinfunction "1")
+			(pintype "input")
+		)
+		(pad "1" thru_hole circle
+			(at 0 2.625)
+			(size 0.8 0.8)
+			(drill 0.5)
+			(layers "*.Cu" "*.Mask")
+			(remove_unused_layers no)
+			(net 9 "Earth")
+			(pinfunction "1")
+			(pintype "input")
+			(zone_connect 2)
+		)
+		(pad "1" thru_hole circle
+			(at 1.856155 -1.856155)
+			(size 0.8 0.8)
+			(drill 0.5)
+			(layers "*.Cu" "*.Mask")
+			(remove_unused_layers no)
+			(net 9 "Earth")
+			(pinfunction "1")
+			(pintype "input")
+			(zone_connect 2)
+		)
+		(pad "1" thru_hole circle
+			(at 1.856155 1.856155)
+			(size 0.8 0.8)
+			(drill 0.5)
+			(layers "*.Cu" "*.Mask")
+			(remove_unused_layers no)
+			(net 9 "Earth")
+			(pinfunction "1")
+			(pintype "input")
+			(zone_connect 2)
+		)
+		(pad "1" thru_hole circle
+			(at 2.625 0)
+			(size 0.8 0.8)
+			(drill 0.5)

Commit message: Revert relays from G2RL-1A-E to G2RL-1A
We really don't need 16A rated relays here, as 12A is already way over
what we're fusing at or plan to support in the power switch connection.

Also decided this time to go with the flux protected 1A model rather
than the fully sealed 1A4 model, because the venting likely helps with
relay life and the relay won't need post-processing steps. Just need to
make sure the board isn't immersed after soldering, but that may related
to other components as well.
Parts:
- K1, K2: footprint lib_fp:Relay_SPST_Omron_G2RL-1A-E -> lib_fp:Relay_SPST_Omron_G2RL-1A
Connections:
- K1 pad 3: LINE -> /ENLG_AC_L
- K1 pad 4: /ENLG_AC_L -> LINE
- K1 pad 5: /ENLG_AC_L -> +12V
- K2 pad 3: LINE -> /SFLT_AC_L
- K2 pad 4: /SFLT_AC_L -> LINE
- K2 pad 5: /SFLT_AC_L -> +12V
Routing:
- net /ENLG_AC_L: track 0.00 -> 21.4 mm
- net /SFLT_AC_L: track 0.00 -> 8.80 mm
- net LINE: track 81.5 -> 80.9 mm
- removed copper zone on B.Cu, net /ENLG_AC_L
- removed copper zone on B.Cu, net /SFLT_AC_L
Changed lines of the file:
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@@
 		)
 	)
-	(footprint "lib_fp:Relay_SPST_Omron_G2RL-1A-E"
+	(footprint "lib_fp:Relay_SPST_Omron_G2RL-1A"
 		(locked yes)
 		(layer "F.Cu")
 		(at 110.25 95 90)
-		(descr "Relay SPST Omron G2RL-1A-E")
-		(tags "Relay SPST Omron G2RL-1A-E")
+		(descr "Relay SPST Omron G2RL-1A")
+		(tags "Relay SPST Omron G2RL-1A")
 		(property "Reference" "K1"
 			(at 12.192 -4.064 90)
@@
 		)
 		(property "Value" "SPST-NO"
-			(at 12.192 7.75 90)
+			(at 12.192 11.43 90)
 			(layer "F.Fab")
 			(effects
@@
 			)
 		)
-		(property "Footprint" "lib_fp:Relay_SPST_Omron_G2RL-1A-E"
+		(property "Footprint" "lib_fp:Relay_SPST_Omron_G2RL-1A"
 			(at 0 0 90)
 			(unlocked yes)
@@
 			)
 		)
-		(property "Description" "RELAY GEN PURPOSE SPST 12A 12V"
-			(at 110.25 95 0)
+		(property "Description" "Omron G2RL low profile power relay, SPST-NO"
+			(at 0 0 90)
+			(unlocked yes)
 			(layer "F.Fab")
 			(hide yes)
@@
 			)
 		)
-		(property "Manufacturer PN" "G2RL-1A4-E DC12"
+		(property "Manufacturer PN" "G2RL-1A DC12"
 			(at 0 0 0)
 			(layer "F.Fab")
@@
 			)
 		)
-		(property "Supplier PN" "Z3083-ND"
+		(property "Supplier PN" "Z140-ND"
 			(at 0 0 0)
 			(layer "F.Fab")
@@
 			)
 		)
-		(pad "1" thru_hole rect
+		(pad "1" thru_hole circle
 			(at 0 7.5 90)
-			(size 2.5 2.5)
+			(size 3 3)
 			(drill 1.3)
 			(layers "*.Cu" "*.Mask")
@@
 		)
 		(pad "3" thru_hole circle
-			(at 20 7.5 90)
-			(size 2.5 2.5)
-			(drill 1.3)
-			(layers "*.Cu" "*.Mask")
-			(remove_unused_layers no)
-			(net 3 "LINE")
-			(pintype "passive")
-		)
-		(pad "4" thru_hole circle
-			(at 25 7.5 90)
-			(size 2.5 2.5)
-			(drill 1.3)
-			(layers "*.Cu" "*.Mask")
-			(remove_unused_layers no)
-			(net 4 "/ENLG_AC_L")
-			(pintype "passive")
-		)
-		(pad "5" thru_hole circle
-			(at 25 0 90)
-			(size 2.5 2.5)
+			(at 23.5 7.5 90)
+			(size 3 3)
 			(drill 1.3)
 			(layers "*.Cu" "*.Mask")
@@
 			(pintype "passive")
 		)
-		(pad "6" thru_hole circle
+		(pad "4" thru_hole circle
 			(at 20 0 90)
-			(size 2.5 2.5)
+			(size 3 3)
 			(drill 1.3)
 			(layers "*.Cu" "*.Mask")
@@
 			(pintype "passive")
 		)
-		(pad "8" thru_hole circle
+		(pad "5" thru_hole circle
 			(at 0 0 90)
-			(size 2.5 2.5)
+			(size 3 3)
 			(drill 1.3)
 			(layers "*.Cu" "*.Mask")
@@
 			(pintype "passive")
 		)
-		(model "${KIPRJMOD}/../library/3dmodels/lib_fp.3dshapes/G2RL-1A-E.step"
+		(model "${KIPRJMOD}/../library/3dmodels/lib_fp.3dshapes/G2RL-1A.step"
 			(offset
 				(xyz 0 -7.5 0)
@@
 		)
 	)
-	(footprint "lib_fp:Relay_SPST_Omron_G2RL-1A-E"
+	(footprint "lib_fp:Relay_SPST_Omron_G2RL-1A"
 		(locked yes)
 		(layer "F.Cu")
 		(at 73.25 95 90)
-		(descr "Relay SPST Omron G2RL-1A-E")
-		(tags "Relay SPST Omron G2RL-1A-E")
+		(descr "Relay SPST Omron G2RL-1A")
+		(tags "Relay SPST Omron G2RL-1A")
 		(property "Reference" "K2"
 			(at 12.192 -4.064 90)
@@
 		)
 		(property "Value" "SPST-NO"
-			(at 12.192 7.75 90)
+			(at 12.192 11.43 90)
 			(layer "F.Fab")
 			(effects
@@
 			)
 		)
-		(property "Footprint" "lib_fp:Relay_SPST_Omron_G2RL-1A-E"
+		(property "Footprint" "lib_fp:Relay_SPST_Omron_G2RL-1A"
 			(at 0 0 90)
 			(unlocked yes)
@@
 			)
 		)
-		(property "Description" "RELAY GEN PURPOSE SPST 12A 12V"
-			(at 73.25 95 0)
+		(property "Description" "Omron G2RL low profile power relay, SPST-NO"
+			(at 0 0 90)
+			(unlocked yes)
 			(layer "F.Fab")
 			(hide yes)
@@
 			)
 		)
-		(property "Manufacturer PN" "G2RL-1A4-E DC12"
+		(property "Manufacturer PN" "G2RL-1A DC12"
 			(at 0 0 0)
 			(layer "F.Fab")
@@
 			)
 		)
-		(property "Supplier PN" "Z3083-ND"
+		(property "Supplier PN" "Z140-ND"
 			(at 0 0 0)
 			(layer "F.Fab")
@@
 			)
 		)
-		(pad "1" thru_hole rect
+		(pad "1" thru_hole circle
 			(at 0 7.5 90)
-			(size 2.5 2.5)
+			(size 3 3)
 			(drill 1.3)
 			(layers "*.Cu" "*.Mask")
@@
 		)
 		(pad "3" thru_hole circle
-			(at 20 7.5 90)
-			(size 2.5 2.5)
-			(drill 1.3)
-			(layers "*.Cu" "*.Mask")
-			(remove_unused_layers no)
-			(net 3 "LINE")
-			(pintype "passive")
-		)
-		(pad "4" thru_hole circle
-			(at 25 7.5 90)
-			(size 2.5 2.5)
-			(drill 1.3)
-			(layers "*.Cu" "*.Mask")
-			(remove_unused_layers no)
-			(net 5 "/SFLT_AC_L")
-			(pintype "passive")
-		)
-		(pad "5" thru_hole circle
-			(at 25 0 90)
-			(size 2.5 2.5)
+			(at 23.5 7.5 90)
+			(size 3 3)
 			(drill 1.3)
 			(layers "*.Cu" "*.Mask")
@@
 			(pintype "passive")
 		)
-		(pad "6" thru_hole circle
+		(pad "4" thru_hole circle
 			(at 20 0 90)
-			(size 2.5 2.5)
+			(size 3 3)
 			(drill 1.3)
 			(layers "*.Cu" "*.Mask")
@@
 			(pintype "passive")
 		)
-		(pad "8" thru_hole circle
+		(pad "5" thru_hole circle
 			(at 0 0 90)
-			(size 2.5 2.5)
+			(size 3 3)
 			(drill 1.3)
 			(layers "*.Cu" "*.Mask")
@@
 			(pintype "passive")
 		)
-		(model "${KIPRJMOD}/../library/3dmodels/lib_fp.3dshapes/G2RL-1A-E.step"
+		(model "${KIPRJMOD}/../library/3dmodels/lib_fp.3dshapes/G2RL-1A.step"
 			(offset
 				(xyz 0 -7.5 0)
@@
 	)
 	(segment
-		(start 110.25 75)
-		(end 117.75 75)
+		(start 99.06 78.486)
+		(end 102.546 75)
 		(width 3.5)
 		(layer "F.Cu")
@@
 	)
 	(segment
-		(start 80.75 75)
-		(end 73.25 75)
+		(start 118.75 83.5)
+		(end 120.25 83.5)
+		(width 3.5)
+		(layer "F.Cu")
+		(net 3)
+	)
+	(segment
+		(start 110.25 75)
+		(end 118.75 83.5)
 		(width 3.5)
 		(layer "F.Cu")
@@
 	)
 	(segment
-		(start 80.75 75)
+		(start 102.546 75)
 		(end 110.25 75)
 		(width 3.5)
@@
 	)
 	(segment
-		(start 117.75 81)
-		(end 120.25 83.5)
+		(start 76.736 78.486)
+		(end 99.06 78.486)
 		(width 3.5)
 		(layer "F.Cu")
@@
 	)
 	(segment
-		(start 117.75 75)
-		(end 117.75 81)
+		(start 73.25 75)
+		(end 76.736 78.486)
 		(width 3.5)
 		(layer "F.Cu")
@@
 	)
 	(segment
+		(start 117.75 71.5)
+		(end 117.75 65.511)
+		(width 3.5)
+		(layer "B.Cu")
+		(net 4)
+	)
+	(segment
+		(start 120.461 62.8)
+		(end 132 62.8)
+		(width 3.5)
+		(layer "B.Cu")
+		(net 4)
+	)
+	(segment
+		(start 117.75 65.511)
+		(end 120.461 62.8)
+		(width 3.5)
+		(layer "B.Cu")
+		(net 4)
+	)
+	(segment
+		(start 80.75 71.5)
+		(end 80.75 63.05)
+		(width 3.5)
+		(layer "B.Cu")
+		(net 5)
+	)
+	(segment
+		(start 80.75 63.05)
+		(end 81 62.8)
+		(width 3.5)
+		(layer "B.Cu")
+		(net 5)
+	)
+	(segment
 		(start 146 57.076)
 		(end 143.407 54.483)
@@
 	)
 	(zone
-		(net 5)
-		(net_name "/SFLT_AC_L")
-		(layer "B.Cu")
-		(hatch edge 0.5)
-		(priority 3)
-		(connect_pads yes
-			(clearance 0.508)
-		)
-		(min_thickness 0.25)
-		(filled_areas_thickness no)
-		(fill yes
-			(thermal_gap 0.5)
-			(thermal_bridge_width 0.5)
-			(smoothing fillet)
-			(radius 2)
-		)
-		(polygon
-			(pts
-				(xy 83 60.5) (xy 79 60.5) (xy 71 67.5) (xy 71 72) (xy 83 72)
-			)
-		)
-	)
-	(zone
 		(net 1)
 		(net_name "GND")
@@
 			)
 		)
-	)
-	(zone
-		(net 4)
-		(net_name "/ENLG_AC_L")
-		(layer "B.Cu")
-		(hatch edge 0.5)
-		(priority 3)
-		(connect_pads yes
-			(clearance 0.508)
-		)
-		(min_thickness 0.25)
-		(filled_areas_thickness no)
-		(fill yes
-			(thermal_gap 0.5)
-			(thermal_bridge_width 0.5)
-			(smoothing fillet)
-			(radius 2)
-		)
-		(polygon
-			(pts
-				(xy 120 66) (xy 121 65) (xy 134 65) (xy 134 60.5) (xy 116 60.5) (xy 108 67.5) (xy 108 72) (xy 120 72)
-			)
-		)

Commit message: Change power switch connector from Mega-Fit to Mini-Fit Jr
This swaps the power connector for a smaller one, and moves it slightly
to resolve mechanical clearance issues. Fixes #52

Some routing cleanup may still be needed, but it'll be done as part of
future changes.
Parts:
- J1: footprint Connector_Molex:Molex_Mega-Fit_76829-0002_2x01_P5.70mm_Vertical -> lib_fp:Molex_Mini-Fit_Jr_172447_2x01_P4.20mm_Vertical
- moved J1 13.1 mm to (128.0, 70.5), turned to 0 degrees
Connections:
- F1 pad 1: Net-(J1-B) -> Net-(J1-A)
- J1 pad 1: LINE -> Net-(J1-A)
- J1 pad 2: Net-(J1-B) -> LINE
Routing:
- net Net-(J1-B): track 52.5 -> 0.00 mm
- net Net-(J1-A): track 0.00 -> 49.4 mm
- net LINE: track 80.9 -> 88.3 mm
Other:
- board text added: "Main Board Overlap"

Commit message: Add filtering components to input of AC/DC converter
Remove the internal fuse and MOV, since they appear to be redundant with
components already inside the sealed AC/DC converter block.

Add AC line filter to the input of the AC/DC converter, to help reduce
problems caused by external line noise.

Standardize on slightly thinner power traces and a 2.5mm clearance rule, to
make sure everything fits.  With 2oz copper, this should still be okay.

Refs #56
Parts:
- removed F2: Fuse, Fuse:Fuseholder_Cylinder-5x20mm_Schurter_0031_8201_Horizontal_Open
- removed RV1: S14K350, lib_fp:RV_Disc_D15.5mm_W5.6mm_P7.5mm
- added C4: 0.1uF(X2), lib_fp:C_Rect_L18.0mm_W5.0mm_P15.00mm_Kemet_R46, F.Cu at (148.5, 86.5)
- added C5: 2200pF(Y1), lib_fp:C_Disc_D12.0mm_W5.0mm_P10.00mm_Vishay_VY1, F.Cu at (177.2, 89.2)
- added C6: 2200pF(Y1), lib_fp:C_Disc_D12.0mm_W5.0mm_P10.00mm_Vishay_VY1, F.Cu at (171.0, 81.5)
- added FL1: 15uH, lib_fp:Choke_Schaffner_RN212-02-12.5x18.0mm, F.Cu at (155.0, 71.5)
Connections:
- PS1 pad 1: NEUT -> /AC_F_N
- PS1 pad 2: /AC_L -> /AC_F_L
Routing:
- net Earth: track 51.6 -> 98.9 mm
- net /AC_F_N: track 0.00 -> 26.9 mm
- net /AC_F_L: track 0.00 -> 22.2 mm
- net NEUT: track 158.7 -> 136.8 mm
- net /AC_L: track 21.1 -> 0.00 mm
- net Net-(J1-A): track 49.4 -> 63.8 mm
- net LINE: track 88.3 -> 96.9 mm
Other:
- board text removed: "Internal Fuse"
